Commit message: Fix collision geometries of allegro hand to prevent self-collisions

File: src/vid2skill/models/franka_allegro/franka_allegro.urdf (robot description, URDF)
Before this commit: robot franka_allegro, 30 links, 29 joints
Links:
- link allegro_link_0: geometry collision box size=0.0196 0.0275 0.0164; visual mesh filename=assets/allegro_hand/link_0.0.gltf
- link allegro_link_1: geometry collision box size=0.0196 0.0275 0.054; visual mesh filename=assets/allegro_hand/link_1.0.gltf
- link allegro_link_10: geometry collision box size=0.0196 0.0275 0.0384; visual mesh filename=assets/allegro_hand/link_2.0.gltf
- link allegro_link_11: geometry collision box size=0.0196 0.0275 0.0267; visual mesh filename=assets/allegro_hand/link_3.0.gltf
- link allegro_link_11_tip: geometry collision sphere radius=0.012; visual mesh filename=assets/allegro_hand/link_3.0_tip.gltf
- link allegro_link_12: geometry collision box size=0.0358 0.034 0.0455; visual mesh filename=assets/allegro_hand/link_12.0_right.gltf
- link allegro_link_13: geometry collision box size=0.0196 0.0275 0.0177; visual mesh filename=assets/allegro_hand/link_13.0.gltf
- link allegro_link_14: geometry collision box size=0.0196 0.0275 0.0514; visual mesh filename=assets/allegro_hand/link_14.0.gltf
- link allegro_link_15: geometry collision box size=0.0196 0.0275 0.0423; visual mesh filename=assets/allegro_hand/link_15.0.gltf
- link allegro_link_15_tip: geometry collision sphere radius=0.012; visual mesh filename=assets/allegro_hand/link_15.0_tip.gltf
- link allegro_link_2: geometry collision box size=0.0196 0.0275 0.0384; visual mesh filename=assets/allegro_hand/link_2.0.gltf
- link allegro_link_3: geometry collision box size=0.0196 0.0275 0.0267; visual mesh filename=assets/allegro_hand/link_3.0.gltf
- link allegro_link_3_tip: geometry collision sphere radius=0.012; visual mesh filename=assets/allegro_hand/link_3.0_tip.gltf
- link allegro_link_4: geometry collision box size=0.0196 0.0275 0.0164; visual mesh filename=assets/allegro_hand/link_0.0.gltf
- link allegro_link_5: geometry collision box size=0.0196 0.0275 0.054; visual mesh filename=assets/allegro_hand/link_1.0.gltf
- link allegro_link_6: geometry collision box size=0.0196 0.0275 0.0384; visual mesh filename=assets/allegro_hand/link_2.0.gltf
- link allegro_link_7: geometry collision box size=0.0196 0.0275 0.0267; visual mesh filename=assets/allegro_hand/link_3.0.gltf
- link allegro_link_7_tip: geometry collision sphere radius=0.012; visual mesh filename=assets/allegro_hand/link_3.0_tip.gltf
- link allegro_link_8: geometry collision box size=0.0196 0.0275 0.0164; visual mesh filename=assets/allegro_hand/link_0.0.gltf
- link allegro_link_9: geometry collision box size=0.0196 0.0275 0.054; visual mesh filename=assets/allegro_hand/link_1.0.gltf
- link allegro_palm_link: geometry collision box size=0.0408 0.0565 0.0475; collision box size=0.0408 0.0565 0.095
- link panda_link7: geometry collision sphere radius=0.05; collision sphere radius=0.052
- link panda_link8: geometry collision box size=0.08 0.08 0.04
